File: PCB/soundcard v1.1.sch (EAGLE design)
At the start: 309 parts, among them IC1 ADP7118, IC10 AD797, IC11 AD797, IC12 AD797, IC13 S34ML, IC14 TPS73801, IC15 USBLC6-2SC6, IC16 PIC32MZ2048EFM100, IC17 USBLC6-2SC6, IC18 LP5907MFX-3.3, IC19 FT232RL, IC2 ADP5070EP, IC20 LP5907MFX-3.3, IC21 SI8642BC-B-IS1, IC22 SN74LVC1G125, IC23 SN74LVC1G125, IC24 SN74LVC1G125, IC25 ATXMEGAxxxA4U-AU, IC26 SI8645, IC27 SN65HVD, IC28 M74VHC1GT50DTT1G, IC29 M74VHC1GT50DTT1G, IC3 ADP7182, IC30 SN74LVC1G125, IC31 SN74LVC1G125, IC32 TPS73801, IC33 VHC1GT126, IC34 VHC1GT126, IC35 VHC1GT125, IC4 ADP3303, IC5 ADP3303, IC6 AD1955, IC7 AD797, IC8 AD797, IC9 AD797, J1 Port 1, J2 Port 1, J3 RCARCA, J4 RCARCA, SW1 SW1", X1 CON_3.5MM_1X10

Commit message: Replaced PCB files with the version 1.1.
Parts:
- added C144, C145: 15nF, rcl:C-EUC0402
- added C146, C147: 100nF, rcl:C-EUC0402
- added C148, C149: 1u, rcl:C-EUC0603
- added IC37, IC38: OPA365, CNP-ics 2:OPA365
- added R80: 3.16k, rcl:R-EU_R0402
- added R81, R82: 10k, rcl:R-EU_R0402
- added R83, R85: 24k, rcl:R-EU_R0402
- added R84, R86: 16k, rcl:R-EU_R0402
- added R87, R88, R89: 100k, rcl:R-EU_R0402
- R78, R79: value 10k -> 100k
- renumbered TX1 to LED1, TX2 to LED2, TX3 to LED3
Connections:
- new net ADC0_IN: R83.2, X1.7
- new net ADC1_IN: R85.2, X1.6
- new net N$19: IC37.-IN, IC37.OUT, R81.1
- new net N$44: IC37.+IN, R83.1, R84.2
- new net N$57: IC38.+IN, R85.1, R86.2
- new net N$6: IC38.-IN, IC38.OUT, R82.1
- new net N$79: C148.1, IC1.EN, R79.1, R87.2
- new net N$83: C149.1, IC3.EN, R78.1, R88.2
- net ADC0: now also C144.2, R81.2; no longer X1.7
- net ADC1: now also C145.2, R82.2; no longer X1.6
- net BUSY: now also R80.1
- net EN_N12V: now also R88.1; no longer IC3.EN, R78.1
- net EN_P12V: now also R87.1; no longer IC1.EN, R79.1
- net GND: now also C144.1, C145.1, C146.2, C147.2, C148.2, C149.2, IC37.V-, IC38.V-, R84.1, R86.1, R89.2
- net UC_IO3: now also R89.1
- net VCC: now also R80.2
- net VCCIO: now also C146.1, C147.1, IC37.V+, IC38.V+
Other:
- note added: "2nd Order LPF: 1.061 kHz"
- note added: "Licensed under the TAPR Open Hardware License (www.tapr.org/OHL) Copyright 2017 Artur Silva and Filipe Carvalho"
- note added: "Licensed under the TAPR Open Hardware License (www.tapr.org/OHL) Copyright 2017-2019 Artur Silva, Dario Bento, Paulo Carriço and Filipe Carvalho"
- note added: "Vmax=5V -> VADCmax=2V (AVCC/1.6)"
- note removed: "Licensed under the TAPR Open Hardware License (www.tapr.org/OHL) Copyright 2018 Artur Silva, Dario Bento, Paulo Carriço, Filipe Carvalho"
- moved on the sheet: JP2, R78, R79, X1
