File: PCB/soundcard v1.1.brd (EAGLE design)
At the start: 152 x 148.5 mm, 311 parts, among them IC1 ADP7118, IC10 AD797, IC11 AD797, IC12 AD797, IC13 S34ML, IC14 TPS73801, IC15 USBLC6-2SC6, IC16 PIC32MZ2048EFM100, IC17 USBLC6-2SC6, IC18 LP5907MFX-3.3, IC19 FT232RL, IC2 ADP5070EP, IC20 LP5907MFX-3.3, IC21 SI8642BC-B-IS1, IC22 SN74LVC1G125, IC23 SN74LVC1G125, IC24 SN74LVC1G125, IC25 ATXMEGAxxxA4U-AU, IC26 SI8645, IC27 SN65HVD, IC28 M74VHC1GT50DTT1G, IC29 M74VHC1GT50DTT1G, IC3 ADP7182, IC30 SN74LVC1G125, IC31 SN74LVC1G125, IC32 TPS73801, IC33 VHC1GT126, IC34 VHC1GT126, IC35 VHC1GT125, IC4 ADP3303, IC5 ADP3303, IC6 AD1955, IC7 AD797, IC8 AD797, IC9 AD797, J1 Port 1, J2 Port 1, J3 RCARCA, J4 RCARCA, SW1 SW1", X1 CON_3.5MM_1X10

Commit message: Replaced PCB files with the version 1.1.
Parts:
- added C144, C145: 15nF, rcl:C0402
- added C146, C147: 100nF, rcl:C0402
- added C148, C149: 1u, rcl:C0603
- added IC37, IC38: OPA365, CNP-ics 2:SOT23-5
- added R80: 3.16k, rcl:R0402
- added R81, R82: 10k, rcl:R0402
- added R83, R85: 24k, rcl:R0402
- added R84, R86: 16k, rcl:R0402
- added R87, R88, R89: 100k, rcl:R0402
- R78, R79: value 10k -> 100k
- moved GND174 1.25 mm to (74.2, 40.5)
- moved R79 0.89 mm to (62.6, 129.6), turned to 270 degrees
- moved C131 0.50 mm to (52.7, 28.6)
- renumbered TX1 to LED1, TX2 to LED2, TX3 to LED3
Connections:
- new net ADC0_IN: R83.2, X1.P7
- new net ADC1_IN: R85.2, X1.P6
- new net N$19: IC37.1, IC37.4, R81.1
- new net N$44: IC37.3, R83.1, R84.2
- new net N$57: IC38.3, R85.1, R86.2
- new net N$6: IC38.1, IC38.4, R82.1
- new net N$79: C148.1, IC1.3, R79.1, R87.2
- new net N$83: C149.1, IC3.3, R78.1, R88.2
- net ADC0: now also C144.2, R81.2; no longer X1.P7
- net ADC1: now also C145.2, R82.2; no longer X1.P6
- net BUSY: now also R80.1
- net EN_N12V: now also R88.1; no longer IC3.3, R78.1
- net EN_P12V: now also R87.1; no longer IC1.3, R79.1
- net GND: now also C144.1, C145.1, C146.2, C147.2, C148.2, C149.2, IC37.2, IC38.2, R84.1, R86.1, R89.2
- net UC_IO3: now also R89.1
- net VCC: now also R80.2
- net VCCIO: now also C146.1, C147.1, IC37.5, IC38.5
Routing:
- net ADC0: track 95.9 -> 43.5 mm
- net ADC1: track 100.9 -> 53.0 mm
- net ADC0_IN: track 0.00 -> 43.8 mm, vias 0 -> 2
- net ADC1_IN: track 0.00 -> 38.9 mm, vias 0 -> 2
- net VCCIO: track 318.8 -> 339.1 mm, vias 16 -> 18
- net N$83: track 0.00 -> 8.17 mm
- net EN_N12V: track 85.2 -> 77.1 mm
- net N$79: track 0.00 -> 7.21 mm
- net N$19: track 0.00 -> 6.08 mm
- net EN_P12V: track 75.7 -> 69.7 mm
- net N$6: track 0.00 -> 5.91 mm
- net N$44: track 0.00 -> 3.66 mm
- net N$57: track 0.00 -> 3.54 mm
- net BUSY: track 63.4 -> 64.7 mm
- net UC_IO3: track 92.8 -> 93.9 mm
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Other:
- board text added: "Licensed under the TAPR Open Hardware License (www.tapr.org/OHL) Copyright 2017-2019 Artur Silva, Dario Bento, Paulo Carriço and Filipe Carvalho"
- board text added: "harp sound card v1.1"
- board text removed: "Licensed under the TAPR Open Hardware License (www.tapr.org/OHL) Copyright 2018 Artur Silva, Dario Bento, Paulo Carriço, Filipe Carvalho"
- board text removed: "sound card v1.0"

Commit message: Minor changes and added gerbers.
Parts:
- moved C25 4.95 mm to (61.5, 128.2)
- moved C1 4.95 mm to (65.5, 136.5)
- moved C9 4.95 mm to (65.3, 143.7)
- moved R71 4.95 mm to (66.4, 68.6)
- moved C121 4.95 mm to (49.5, 32.6)
- moved C130 4.95 mm to (59.3, 33.1)
- moved IC18 4.95 mm to (34.6, 88.7)
- moved J1 4.95 mm to (35.4, 7.90)
- moved OSC2 4.95 mm to (52.6, 32.6)
- moved PDI 4.95 mm to (66.0, 32.4)
- moved R69 4.95 mm to (89.6, 33.2)
- moved C17 4.95 mm to (16.5, 125.0)
- moved D2 4.95 mm to (9.65, 121.3)
- moved IC15 4.95 mm to (9.90, 92.1)
- moved IC17 4.95 mm to (17.4, 48.4)
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